File: Ethernet.kicad_sch (KiCad schematic)
At the start: 47 parts, among them J10 Conn_01x06, J11 Conn_01x06, J12 Conn_01x06, J8 ARJM11B1-009-AB-EW2, J9 Conn_01x06, U8 W5500, Y1 ABM8-25.000MHZ-B2Y-T

Commit message: Add information on PCB and schematic
Other:
- company: (none) -> KN NaMi
- title: (none) -> Ethernet
Changed lines of the file:
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@@
 	(generator_version "9.0")
 	(paper "A4")
+	(title_block
+		(title "Ethernet")
+		(date "2025-12-22")
+		(rev "0.0.1")
+		(company "KN NaMi")
+	)
 	(text "20,32mm"
 		(exclude_from_sim no)
