File: Power supplay.kicad_sch (KiCad schematic)
At the start: 55 parts, among them J1 DC_12V_IN, J2 GND, J3 Conn_02x07, U1 MC7805BDTRKG, U2 LD1117AS33TR, U3 LTC3260xMSE, U4 TL431AIL5T, U5 REF3033, U6 TL431

Commit message: Add information on PCB and schematic
Other:
- company: (none) -> KN NaMi
- title: (none) -> power supplay
Changed lines of the file:
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@@
 	(generator_version "9.0")
 	(paper "A4")
+	(title_block
+		(title "power supplay")
+		(date "2025-12-22")
+		(rev "0.0.1")
+		(company "KN NaMi")
+	)
 	(text "V_ka = V_ref*(1+R1/R2)+R1*I_ref\nV_ka = 2.495*(1+1000/10000)+1000*1,8*10^(-6)\nV_ka = 2,7463 V\n\nI_out = V_ka/330\nI_out = (12-2,7463)/330\nI_out = 28 mA"
 		(exclude_from_sim no)
@@
 			(width 0)
 			(type default)
+		)
+	)
+	(table
+		(column_count 2)
+		(border
+			(external yes)
+			(header yes)
+			(stroke
+				(width 0)
+				(type solid)
+			)
+		)
+		(separators
+			(rows yes)
+			(cols yes)
+			(stroke
+				(width 0)
+				(type solid)
+			)
+		)
+		(column_widths 41.275 27.305)
+		(row_heights 3.175 3.175 3.175 3.175 3.175)
+		(cells
+			(table_cell "Output Voltage"
+				(exclude_from_sim no)
+				(at 81.28 130.175 0)
+				(size 41.275 3.175)
+				(margins 0.9525 0.9525 0.9525 0.9525)
+				(span 1 1)
+				(fill
+					(type none)
+				)
+				(effects
+					(font
+						(size 1.27 1.27)
+					)
+					(justify left top)
+				)
+			)
+			(table_cell "3.3"
+				(exclude_from_sim no)
+				(at 122.555 130.175 0)
+				(size 27.305 3.175)
+				(margins 0.9525 0.9525 0.9525 0.9525)
+				(span 1 1)
+				(fill
+					(type none)
+				)
+				(effects
+					(font
+						(size 1.27 1.27)
+					)
+					(justify left top)
+				)
+			)
+			(table_cell "Load curren specification for REF30xx"
+				(exclude_from_sim no)
+				(at 81.28 133.35 0)
+				(size 41.275 3.175)
+				(margins 0.9525 0.9525 0.9525 0.9525)
+				(span 1 1)
+				(fill
+					(type none)
+				)
+				(effects
+					(font
+						(size 1.27 1.27)
+					)
+					(justify left top)
+				)
+			)
+			(table_cell "max 25 mA"
+				(exclude_from_sim no)
+				(at 122.555 133.35 0)
+				(size 27.305 3.175)
+				(margins 0.9525 0.9525 0.9525 0.9525)
+				(span 1 1)
+				(fill
+					(type none)
+				)
+				(effects
+					(font
+						(size 1.27 1.27)
+					)
+					(justify left top)
+				)
+			)
+			(table_cell "Load curren specification for REF30xxE"
+				(exclude_from_sim no)
+				(at 81.28 136.525 0)
+				(size 41.275 3.175)
+				(margins 0.9525 0.9525 0.9525 0.9525)
+				(span 1 1)
+				(fill
+					(type none)
+				)
+				(effects
+					(font
+						(size 1.27 1.27)
+					)
+					(justify left top)
+				)
+			)
+			(table_cell "min -10 mA max 10 mA"
+				(exclude_from_sim no)
+				(at 122.555 136.525 0)
+				(size 27.305 3.175)
+				(margins 0.9525 0.9525 0.9525 0.9525)
+				(span 1 1)
+				(fill
+					(type none)
+				)
+				(effects
+					(font
+						(size 1.27 1.27)
+					)
+					(justify left top)
+				)
+			)
+			(table_cell "Initial accuracy for REF30xx"
+				(exclude_from_sim no)
+				(at 81.28 139.7 0)
+				(size 41.275 3.175)
+				(margins 0.9525 0.9525 0.9525 0.9525)
+				(span 1 1)
+				(fill
+					(type none)
+				)
+				(effects
+					(font
+						(size 1.27 1.27)
+					)
+					(justify left top)
+				)
+			)
+			(table_cell "0,2%"
+				(exclude_from_sim no)
+				(at 122.555 139.7 0)
+				(size 27.305 3.175)
+				(margins 0.9525 0.9525 0.9525 0.9525)
+				(span 1 1)
+				(fill
+					(type none)
+				)
+				(effects
+					(font
+						(size 1.27 1.27)
+					)
+					(justify left top)
+				)
+			)
+			(table_cell "Initial accuracy for REF30xxE"
+				(exclude_from_sim no)
+				(at 81.28 142.875 0)
+				(size 41.275 3.175)
+				(margins 0.9525 0.9525 0.9525 0.9525)
+				(span 1 1)
+				(fill
+					(type none)
+				)
+				(effects
+					(font
+						(size 1.27 1.27)
+					)
+					(justify left top)
+				)
+			)
+			(table_cell "0,1%"
+				(exclude_from_sim no)
+				(at 122.555 142.875 0)
+				(size 27.305 3.175)
+				(margins 0.9525 0.9525 0.9525 0.9525)
+				(span 1 1)
+				(fill
+					(type none)
+				)
+				(effects
+					(font
+						(size 1.27 1.27)
+					)
+					(justify left top)
+				)
+			)
 		)
 	)
@@
 				(margins 0.9525 0.9525 0.9525 0.9525)
 				(span 1 1)
-				(fill
-					(type none)
-				)
-				(effects
-					(font
-						(size 1.27 1.27)
-					)
-					(justify left top)
-				)
-			)
-		)
-	)
-	(table
-		(column_count 2)
-		(border
-			(external yes)
-			(header yes)
-			(stroke
-				(width 0)
-				(type solid)
-			)
-		)
-		(separators
-			(rows yes)
-			(cols yes)
-			(stroke
-				(width 0)
-				(type solid)
-			)
-		)
-		(column_widths 41.275 27.305)
-		(row_heights 3.175 3.175 3.175 3.175 3.175)
-		(cells
-			(table_cell "Output Voltage"
-				(exclude_from_sim no)
-				(at 81.28 130.175 0)
-				(size 41.275 3.175)
-				(margins 0.9525 0.9525 0.9525 0.9525)
-				(span 1 1)
-				(fill
-					(type none)
-				)
-				(effects
-					(font
-						(size 1.27 1.27)
-					)
-					(justify left top)
-				)
-			)
-			(table_cell "3.3"
-				(exclude_from_sim no)
-				(at 122.555 130.175 0)
-				(size 27.305 3.175)
-				(margins 0.9525 0.9525 0.9525 0.9525)
-				(span 1 1)
-				(fill
-					(type none)
-				)
-				(effects
-					(font
-						(size 1.27 1.27)
-					)
-					(justify left top)
-				)
-			)
-			(table_cell "Load curren specification for REF30xx"
-				(exclude_from_sim no)
-				(at 81.28 133.35 0)
-				(size 41.275 3.175)
-				(margins 0.9525 0.9525 0.9525 0.9525)
-				(span 1 1)
-				(fill
-					(type none)
-				)
-				(effects
-					(font
-						(size 1.27 1.27)
-					)
-					(justify left top)
-				)
-			)
-			(table_cell "max 25 mA"
-				(exclude_from_sim no)
-				(at 122.555 133.35 0)
-				(size 27.305 3.175)
-				(margins 0.9525 0.9525 0.9525 0.9525)
-				(span 1 1)
-				(fill
-					(type none)
-				)
-				(effects
-					(font
-						(size 1.27 1.27)
-					)
-					(justify left top)
-				)
-			)
-			(table_cell "Load curren specification for REF30xxE"
-				(exclude_from_sim no)
-				(at 81.28 136.525 0)
-				(size 41.275 3.175)
-				(margins 0.9525 0.9525 0.9525 0.9525)
-				(span 1 1)
-				(fill
-					(type none)
-				)
-				(effects
-					(font
-						(size 1.27 1.27)
-					)
-					(justify left top)
-				)
-			)
-			(table_cell "min -10 mA max 10 mA"
-				(exclude_from_sim no)
-				(at 122.555 136.525 0)
-				(size 27.305 3.175)
-				(margins 0.9525 0.9525 0.9525 0.9525)
-				(span 1 1)
-				(fill
-					(type none)
-				)
-				(effects
-					(font
-						(size 1.27 1.27)
-					)
-					(justify left top)
-				)
-			)
-			(table_cell "Initial accuracy for REF30xx"
-				(exclude_from_sim no)
-				(at 81.28 139.7 0)
-				(size 41.275 3.175)
-				(margins 0.9525 0.9525 0.9525 0.9525)
-				(span 1 1)
-				(fill
-					(type none)
-				)
-				(effects
-					(font
-						(size 1.27 1.27)
-					)
-					(justify left top)
-				)
-			)
-			(table_cell "0,2%"
-				(exclude_from_sim no)
-				(at 122.555 139.7 0)
-				(size 27.305 3.175)
-				(margins 0.9525 0.9525 0.9525 0.9525)
-				(span 1 1)
-				(fill
-					(type none)
-				)
-				(effects
-					(font
-						(size 1.27 1.27)
-					)
-					(justify left top)
-				)
-			)
-			(table_cell "Initial accuracy for REF30xxE"
-				(exclude_from_sim no)
-				(at 81.28 142.875 0)
-				(size 41.275 3.175)
-				(margins 0.9525 0.9525 0.9525 0.9525)
-				(span 1 1)
-				(fill
-					(type none)
-				)
-				(effects
-					(font
-						(size 1.27 1.27)
-					)
-					(justify left top)
-				)
-			)
-			(table_cell "0,1%"
-				(exclude_from_sim no)
-				(at 122.555 142.875 0)
-				(size 27.305 3.175)
-				(margins 0.9525 0.9525 0.9525 0.9525)
-				(span 1 1)
