File: STM_proto_board.kicad_sch (KiCad schematic)
At the start: 0 parts

Commit message: Add information on PCB and schematic
Other:
- company: (none) -> KN NaMi
- title: (none) -> main schematic
Changed lines of the file:
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@@
 	(generator_version "9.0")
 	(paper "A4")
+	(title_block
+		(title "main schematic")
+		(date "2025-12-22")
+		(rev "0.0.1")
+		(company "KN NaMi")
+	)
 	(text_box "- wzmacniacze odwracające, nieodwracające, różnicowe,\n- pomiar prądu,\n- filtry aktywne,\n- wzmacniasz operacyjny robiący konwersję z 0V - 3.3V na -12V - 12V,\n- wzmacniacz w drugą stronę,\n- bufor na wyjściu,"
 		(exclude_from_sim no)
