File: The rest of the things.kicad_sch (KiCad schematic)
At the start: 92 parts, among them J13 pot, J14 i2c adafruit, J15 SM04B-SRSS-TB, J16 Conn_01x03, J17 AVR-ICSP, J18 Conn_01x03, J19 LED, J20 LOW, J21 HIGH, J22 sw, J23 B6252H5-NPP3G-50, J24 Conn_02x07, J25 Conn_02x07, J26 Conn_02x07, J27 B6252H5-NPP3G-50, J28 Conn_01x06, J29 Conn_01x06, J31 B6252H5-NPP3G-50, J32 B6252H5-NPP3G-50, J33 Conn_02x07, J34 Conn_02x07, J35 Conn_02x07, J36 B6252H5-NPP3G-50, J37 OLED, J38 i2c OLED, J39 ROT_ENC_SW, J40 sw, J41 sw, Q1 BSS138, Q2 BSS138, Q3 BSS138, Q4 BSS138, Q5 BSS138, SW1 SW_Push, SW2 SW_Push, SW3 SW_Push, SW4 SW_Push, SW5 SW_Push, SW6 RotaryEncoder_Switch

Commit message: Add information on PCB and schematic
Other:
- company: (none) -> KN NaMi
- title: (none) -> rest of the things
Changed lines of the file:
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@@
 	(generator_version "9.0")
 	(paper "A3")
+	(title_block
+		(title "rest of the things")
+		(date "2025-12-22")
+		(rev "0.0.1")
+		(company "KN NaMi")
+	)
 	(text "Low Pass Filter"
 		(exclude_from_sim no)
