File: uC.kicad_sch (KiCad schematic)
At the start: 13 parts, among them J4 Conn_01x20, J5 Conn_01x20, J6 Conn_02x12_Odd_Even, J7 Conn_02x12_Odd_Even, U7 STM32G474CoreBoard

Commit message: Add information on PCB and schematic
Other:
- company: (none) -> KN NaMi
- title: (none) -> uC
Changed lines of the file:
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@@
 	(generator_version "9.0")
 	(paper "A3")
+	(title_block
+		(title "uC")
+		(date "2025-12-22")
+		(rev "0.0.1")
+		(company "KN NaMi")
+	)
 	(text_box "- pipico\n- STM32G474 Core Board"
 		(exclude_from_sim no)
